Commit message: fixed laser scanner issues + added laser visualization in RVIZ

File: sjtu_drone_description/urdf/sjtu_drone.urdf (robot description, URDF)
Before this commit: robot sjtu_drone, 5 links, 4 joints
Links:
- added link laser_link
- link base_link: geometry collision mesh filename=file:///home/karan/MyWorkspace/ros2_ws/install/sjtu_drone_d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; visual mesh filename=file:///home/karan/MyWorkspace/ros2_ws/install/sjtu_drone_d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
Joints:
- added joint laser_joint: type fixed, parent base_link, child laser_link, origin xyz=0.2 0 0 rpy=0 0 0

File: sjtu_drone_description/urdf/sjtu_drone.urdf.xacro (robot description, xacro)
@@ -48,4 +48,10 @@
   </joint>
   <link name="front_cam_link"/>
+  <joint name="laser_joint" type="fixed">
+    <origin rpy="0 0 0" xyz="0.2 0 0"/>
+    <parent link="base_link" />
+    <child link="laser_link" />
+  </joint>
+  <link name="laser_link"/>
   <joint name="bottom_cam_joint" type="fixed">
     <origin rpy="0 ${M_PI/2} 0" xyz="0 0 0"/>
@@ -60,5 +66,6 @@
         <remapping>cmd_vel:=cmd_vel</remapping>
         <remapping>imu:=imu</remapping>
-        <remapping>laser_scanner:=laser_scanner</remapping>
+        <remapping>sonar:=sonar</remapping>
+        <remapping>laser_scanner_plugin:=laser_scanner_plugin</remapping>
         <remapping>camera_front:=camera_front</remapping>
         <remapping>camera_bottom:=camera_bottom</remapping>
@@ -129,4 +136,47 @@
   <!-- Sonar sensor in 100fps -->
   <gazebo reference="sonar_link">
+    <sensor name="sonar" type="ray">
+      <always_on>1</always_on>
+      <visualize>1</visualize>
+      <update_rate>30</update_rate>
+      <ray>
+        <scan>
+          <horizontal>
+            <samples>5</samples>
+            <resolution>1.000000</resolution>
+            <min_angle>-0.12</min_angle>
+            <max_angle>0.12</max_angle>
+          </horizontal>
+          <vertical>
+            <samples>5</samples>
+            <resolution>1.000000</resolution>
+            <min_angle>-0.12</min_angle>
+            <max_angle>0.12</max_angle>
+          </vertical>
+        </scan>
+        <range>
+          <min>0.02</min>
+          <max>10</max>
+          <resolution>0.01</resolution>
+        </range>
+        <noise>
+          <type>gaussian</type>
+          <mean>0.0</mean>
+          <stddev>0.01</stddev>
+        </noise>
+      </ray>
+      <plugin name="sonar" filename="libgazebo_ros_ray_sensor.so">
+        <ros>
+          <namespace>${mp['namespace']}</namespace>
+          <!-- <remapping>~/out:=sonar</remapping> -->
+        </ros>
+        <frame_name>${mp['namespace']}/sonar_link</frame_name>
+        <output_type>sensor_msgs/Range</output_type>
+        <radiation_type>ultrasound</radiation_type>
+      </plugin>
+    </sensor>
+  </gazebo>
+  <!-- Laser sensor in 100fps -->
+  <gazebo reference="laser_link">
       <sensor name="laser_scanner" type="ray">
           <always_on>1</always_on>
@@ -153,9 +203,9 @@
               </noise>
           </ray>
-          <plugin name="laser_scanner_plugin" filename="libgazebo_ros_laser.so">
+          <plugin name="laser_scanner" filename="libgazebo_ros_ray_sensor.so">
               <ros>
                   <namespace>${mp['namespace']}</namespace>
               </ros>
-              <frame_name>${mp['namespace']}/sonar_link</frame_name>
+              <frame_name>${mp['namespace']}/laser_link</frame_name>
               <output_type>sensor_msgs/LaserScan</output_type>
               <topicName>scan</topicName> <!-- Adjust as needed -->
